File: executable/schematics/pcb/74hc165 extension board.brd (EAGLE design)
At the start: 8 parts

Commit message: pcb design
Parts:
- added E$10, E$9: (no value), con-lstb:MA03-1
- added E$11: (no value), con-lstb:MA05-1
- added E$12: (no value), con-lstb:MA04-1
- added E$13: (no value), con-wago-500:W237-102
- added E$14: (no value), diode:DO34-7
- E$4: device con-molex:70543-17 -> diode:DO34-7
- moved E$4 31.4 mm to (24.1, 52.1), turned to 90 degrees
- moved E$3 1.27 mm to (44.5, 38.1)
Connections:
- new net S$21: E$14.C, E$3.2, E$9.1, E$9.2, E$9.3
- new net S$22: E$10.1, E$10.2, E$10.3, E$3.3, E$4.C
- new net S$23: E$11.1, E$11.2, E$11.3, E$11.4, E$11.5, E$13.1, E$3.1
- net S$19: now also E$12.1, E$12.2, E$12.3, E$12.4, E$13.2, E$14.A, E$4.A
Routing:
- net S$23: track 0.00 -> 25.4 mm
- net S$19: track 61.4 -> 79.7 mm
- net S$21: track 0.00 -> 10.7 mm
- net S$22: track 0.00 -> 10.7 mm
- net S$20: track 55.0 -> 65.0 mm
- net S$1: track 51.9 -> 50.7 mm
- net S$9: track 53.7 -> 52.5 mm
- net S$8: track 23.0 -> 21.7 mm
- net S$7: track 21.9 -> 20.6 mm
- net S$6: track 21.9 -> 20.6 mm
- net S$5: track 21.9 -> 20.6 mm
- net S$4: track 9.42 -> 8.15 mm
- net S$3: track 20.1 -> 18.8 mm
- net S$2: track 45.8 -> 44.5 mm
- net S$17: track 18.8 -> 17.6 mm
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