File: executable/schematics/pcb/new design/74hc165 extension board.brd (EAGLE design)
At the start: 17 parts

Commit message: new design complete
Parts:
- removed E$10, E$9: (no value), con-lstb:MA03-1
- removed E$11: (no value), con-lstb:MA05-1
- removed E$12: (no value), con-lstb:MA04-1
- removed E$13: (no value), con-wago-500:W237-102
- added E$18, E$19: (no value), diode:DO34-7
- moved E$17 1.27 mm to (62.2, 71.1)
Connections:
- new net S$28: E$19.A, E$3.1
- net S$17: now also E$18.C
- net S$18: now also E$18.A, E$19.C
Routing:
- net S$28: track 0.00 -> 76.5 mm
- net S$18: track 20.6 -> 36.4 mm
- net S$21: track 128.3 -> 137.8 mm
- net S$17: track 21.4 -> 25.2 mm
- net S$22: track 74.3 -> 78.1 mm
- net S$20: track 71.2 -> 74.5 mm
- net S$27: track 70.6 -> 71.1 mm
